Commit message: Change front caster joint and back caster joint to continuous

File: my_rb1_description/urdf/my_rb1_robot.urdf (robot description, URDF)
Before this commit: robot my_rb1_robot, 7 links, 6 joints
Joints:
- joint back_caster_joint: type fixed -> continuous
- joint front_caster_joint: type fixed -> continuous
